File: unicorne-choc.kicad_pcb (KiCad board)
At the start: 2 copper layers, 299.9 x 118.8 mm, 167 parts, among them J1 Battery, J2 TPS43, J3 Expansion, J4 GPIO, J5 PAW3395 / PMW3360, Q1 AO3401A, Q2 2N7002, SW1 R0C0, SW10 R1C3, SW11 R1C4, SW12 R1C5, SW13 R2C0, SW14 R2C1, SW15 R2C2, SW16 R2C3, SW17 R2C4, SW18 R2C5, SW19 R0C6, SW2 R0C1, SW20 R1C6, SW21 R2C6, SW22 R3C0, SW23 R3C1, SW24 R3C2, SW25 R3C3, SW26 R3C4, SW27 R3C5, SW28 R4C0, SW29 R4C1, SW3 R0C2, SW30 R4C2, SW31 R4C3, SW32 R4C4, SW33 R4C5, SW34 R5C0, SW35 R5C1, SW36 R5C2, SW37 R5C3, SW38 R5C4, SW39 R5C5, SW4 R0C3, SW40 R3C6, SW41 R4C6, SW42 R5C6, SW43 Power, SW44 Reset, SW5 R0C4, SW6 R0C5, SW7 R1C0, SW8 R1C1, SW9 R1C2, U1 nice!nano v2

Commit message: Rework LED power, break lines and centre placement; add routing tools
- LED supply chosen by solder jumper JP2: nice!nano VCC, or an external
  supply on new LED IN pads (J6); never the battery pin. SN74LV1T125
  level shifter (U2) with bypass jumper JP3.
- Centre parts rearranged so the nice!nano's matrix pins are clear.
- 0805 hand-solder passives; LED chain runs left to right per row.
- Break lines: no sliver slots, perforated end to end, tabs over the lanes.
- Mounting holes stay inside the board and off the routing lanes.
- Routing tools (lanes, Freerouting driver, maze router) and placeholder
  STEP models. Boards are committed placed but unrouted.

Co-Authored-By: Claude Opus 5.5 <noreply@anthropic.com>
Parts:
- added C2: 100nF, Capacitor_SMD:C_0805_2012Metric_Pad1.18x1.45mm_HandSolder, B.Cu at (201.5, 59.2)
- added J6: LED power in, Connector_PinHeader_2.54mm:PinHeader_1x02_P2.54mm_Vertical, F.Cu at (188.0, 132.3)
- added JP2: LED source, Jumper:SolderJumper-3_P1.3mm_Open_RoundedPad1.0x1.5mm, B.Cu at (202.1, 75.7)
- added JP3: U2 bypass, Jumper:SolderJumper-2_P1.3mm_Open_RoundedPad1.0x1.5mm, B.Cu at (202.0, 68.2)
- added U2: SN74LV1T125, Package_TO_SOT_SMD:SOT-23-5_HandSoldering, B.Cu at (201.5, 63.6)
- C1: footprint Capacitor_SMD:C_0805_2012Metric -> Capacitor_SMD:C_0805_2012Metric_Pad1.18x1.45mm_HandSolder
- R1, R2, R3, R4, R5: footprint Resistor_SMD:R_0603_1608Metric -> Resistor_SMD:R_0805_2012Metric_Pad1.20x1.40mm_HandSolder
- moved LED31 76.0 mm to (215.6, 71.5)
- moved LED35 76.0 mm to (289.3, 52.8)
- moved LED18 76.0 mm to (65.5, 71.1)
- moved LED22 76.0 mm to (139.2, 89.7)
- moved LED41 76.0 mm to (226.1, 108.0)
- moved LED45 76.0 mm to (299.8, 89.3)
- moved LED32 38.0 mm to (233.2, 63.9)
- moved LED34 38.0 mm to (269.7, 53.5)
- moved LED42 38.0 mm to (243.7, 100.5)
- moved LED44 38.0 mm to (280.2, 90.0)
- moved LED19 38.0 mm to (85.0, 71.7)
- moved LED21 38.0 mm to (121.6, 82.2)
- moved Q2 34.6 mm to (198.0, 67.7)
- moved Q1 33.1 mm to (198.0, 75.7)
- moved C1 33.0 mm to (198.0, 83.7)
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Connections:
- JP1 pad 2: LED_DIN -> /LED_DATA
- Q1 pad 2: /VBAT -> /LED_SRC
- R1 pad 1: /VBAT -> /LED_SRC
Other:
- outline, holes or cut-outs redrawn
- board text added: "EXT"
- board text added: "LED IN"
- board text added: "V+"

Commit message: Route the Choc board
lanes.py now has per-switch-type lane layouts. Choc: rows run above the
sockets (y -8.0), reached from each cathode by a short top-layer hop
between the switch holes; LED data and supply below the diode; where the
next column sits lower the row lane jogs on the top layer. Break-line
tabs and mounting-hole keep-outs follow the lanes, and finish_route.py
nudges any hole the lanes still touch and retries failed connections
first. MX routing is unchanged.

DRC (Choc): 0 unconnected, 0 copper violations.

Co-Authored-By: Claude Opus 5.5 <noreply@anthropic.com>
Parts:
- LED10, LED11, LED12, LED7, LED8, LED9: value SK6812MINI -> SK6812MINI-E; footprint LED_SMD:LED_SK6812MINI_PLCC4_3.5x3.5mm_P1.75mm -> LED_SMD:LED_SK6812MINI-E_3.2x2.8mm_P1.5mm_ReverseMount
- LED43, LED44, LED45, LED46, LED47, LED48: value SK6812MINI-E -> SK6812MINI; footprint LED_SMD:LED_SK6812MINI-E_3.2x2.8mm_P1.5mm_ReverseMount -> LED_SMD:LED_SK6812MINI_PLCC4_3.5x3.5mm_P1.75mm
- moved LED51 276.1 mm to (318.0, 84.1), turned to 16 degrees
- moved LED54 276.1 mm to (42.0, 84.1), turned to -16 degrees
- moved LED50 265.6 mm to (312.8, 65.8), turned to 16 degrees
- moved LED53 265.6 mm to (47.2, 65.8), turned to -16 degrees
- moved LED49 255.1 mm to (307.6, 47.6), turned to 16 degrees
- moved LED52 255.1 mm to (52.4, 47.6), turned to -16 degrees
- moved LED7 195.1 mm to (70.7, 52.8), turned to -16 degrees
- moved LED12 162.3 mm to (65.5, 71.1), turned to -16 degrees
- moved LED8 156.7 mm to (90.3, 53.5), turned to -16 degrees
- moved LED10 144.7 mm to (126.8, 63.9), turned to -16 degrees
- moved LED30 130.1 mm to (250.8, 56.4), turned to 16 degrees
- moved LED29 128.4 mm to (233.2, 63.9), turned to 16 degrees
- moved LED26 125.9 mm to (239.9, 124.7), turned to 31 degrees
- moved LED27 124.6 mm to (258.2, 116.7), turned to 16 degrees
- moved LED28 122.5 mm to (215.6, 71.5), turned to 16 degrees
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Connections:
- LED10 pad 1: /LEDs/LED_D10 -> GND
- LED10 pad 2: GND -> /LEDs/LED_D9
- LED10 pad 3: /LEDs/LED_D9 -> LED_VDD
- LED10 pad 4: LED_VDD -> /LEDs/LED_D10
- LED11 pad 1: /LEDs/LED_D11 -> GND
- LED11 pad 2: GND -> /LEDs/LED_D10
- LED11 pad 3: /LEDs/LED_D10 -> LED_VDD
- LED11 pad 4: LED_VDD -> /LEDs/LED_D11
- LED12 pad 1: /LEDs/LED_D12 -> GND
- LED12 pad 2: GND -> /LEDs/LED_D11
- LED12 pad 3: /LEDs/LED_D11 -> LED_VDD
- LED12 pad 4: LED_VDD -> /LEDs/LED_D12
- LED43 pad 1: GND -> /LEDs/LED_D43
- LED43 pad 2: /LEDs/LED_D42 -> GND
- LED43 pad 3: LED_VDD -> /LEDs/LED_D42
- LED43 pad 4: /LEDs/LED_D43 -> LED_VDD
- LED44 pad 1: GND -> /LEDs/LED_D44
- LED44 pad 2: /LEDs/LED_D43 -> GND
- LED44 pad 3: LED_VDD -> /LEDs/LED_D43
- LED44 pad 4: /LEDs/LED_D44 -> LED_VDD
- LED45 pad 1: GND -> /LEDs/LED_D45
- LED45 pad 2: /LEDs/LED_D44 -> GND
- LED45 pad 3: LED_VDD -> /LEDs/LED_D44
- LED45 pad 4: /LEDs/LED_D45 -> LED_VDD
- LED46 pad 1: GND -> /LEDs/LED_D46
- LED46 pad 2: /LEDs/LED_D45 -> GND
- LED46 pad 3: LED_VDD -> /LEDs/LED_D45
- LED46 pad 4: /LEDs/LED_D46 -> LED_VDD
- LED47 pad 1: GND -> /LEDs/LED_D47
- LED47 pad 2: /LEDs/LED_D46 -> GND
- LED47 pad 3: LED_VDD -> /LEDs/LED_D46
- LED47 pad 4: /LEDs/LED_D47 -> LED_VDD
- LED48 pad 1: GND -> /LEDs/LED_D48
- LED48 pad 2: /LEDs/LED_D47 -> GND
- LED48 pad 3: LED_VDD -> /LEDs/LED_D47
- LED48 pad 4: /LEDs/LED_D48 -> LED_VDD
- LED7 pad 1: /LEDs/LED_D7 -> GND
- LED7 pad 2: GND -> /LEDs/LED_D6
- LED7 pad 3: /LEDs/LED_D6 -> LED_VDD
- LED7 pad 4: LED_VDD -> /LEDs/LED_D7
- LED8 pad 1: /LEDs/LED_D8 -> GND
- LED8 pad 2: GND -> /LEDs/LED_D7
- LED8 pad 3: /LEDs/LED_D7 -> LED_VDD
- LED8 pad 4: LED_VDD -> /LEDs/LED_D8
- LED9 pad 1: /LEDs/LED_D9 -> GND
- LED9 pad 2: GND -> /LEDs/LED_D8
- LED9 pad 3: /LEDs/LED_D8 -> LED_VDD
- LED9 pad 4: LED_VDD -> /LEDs/LED_D9
Routing:
- net GND: track 0.00 -> 1954.1 mm, vias 0 -> 256
- net LED_VDD: track 0.00 -> 1031.6 mm, vias 0 -> 27
- net COL0: track 0.00 -> 397.0 mm, vias 0 -> 19
- net COL1: track 0.00 -> 351.0 mm, vias 0 -> 12
- net /LEDs/LED_D51: track 0.00 -> 321.9 mm, vias 0 -> 16
- net COL2: track 0.00 -> 307.8 mm, vias 0 -> 12
- net ROW3: track 0.00 -> 297.1 mm, vias 0 -> 22
- net ROW0: track 0.00 -> 273.8 mm, vias 0 -> 21
- net COL3: track 0.00 -> 268.8 mm, vias 0 -> 10
- net ROW5: track 0.00 -> 266.6 mm, vias 0 -> 20
- net ROW1: track 0.00 -> 263.9 mm, vias 0 -> 18
- net ROW4: track 0.00 -> 258.4 mm, vias 0 -> 22
- net ROW2: track 0.00 -> 250.0 mm, vias 0 -> 17
- net COL4: track 0.00 -> 212.3 mm, vias 0 -> 13
- net COL6: track 0.00 -> 205.8 mm, vias 0 -> 10
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- added copper zone on B.Cu, net GND
- added copper zone on F.Cu, net GND
Other:
- outline, holes or cut-outs redrawn

Commit message: Add 3D models and STEP export
Project footprints point at models in lib/3d/: Kailh MX and Choc hotswap
sockets and the Choc V1 switch (keyswitch-kicad-library), plus placeholder
boxes for the nice!nano, TPS43, MX switch, SK6812MINI and MSK-12C02 (the
last two copied from the stock library with a model added). The trackpad
model sits on a board-only footprint; bare pads carry no model.
export_3d.py writes export/unicorne-{mx,choc}.step; renders alongside.

Both boards regenerated and re-routed: DRC 0 unconnected, 0 copper
violations.

Co-Authored-By: Claude Opus 5.5 <noreply@anthropic.com>
Parts:
- added TP1: TPS43, , F.Cu at (180.0, 101.1)
- LED1, LED2, LED3, LED4, LED43, LED44, LED45, LED46, LED47, LED48, LED5, LED6: footprint LED_SMD:LED_SK6812MINI_PLCC4_3.5x3.5mm_P1.75mm -> unicorne:LED_SK6812MINI_PLCC4_3.5x3.5mm_P1.75mm
- SW43: footprint Button_Switch_SMD:SW_SPDT_Shouhan_MSK12C02 -> unicorne:SW_SPDT_Shouhan_MSK12C02
Routing:
- net GND: track 1954.1 -> 2002.2 mm, vias 256 -> 257
- net /LEDs/LED_D51: track 321.9 -> 353.5 mm, vias 16 -> 6
- net /BATT+: track 86.7 -> 94.2 mm, vias 5 -> 6
- net ROW2: track 250.0 -> 256.9 mm
- net LED_VDD: track 1031.6 -> 1026.4 mm
- net /SDA_MOSI: track 86.6 -> 83.7 mm
- net COL1: track 351.0 -> 348.8 mm, vias 12 -> 11
- net /LEDs/LED_D16: track 94.9 -> 92.7 mm, vias 2 -> 4
- net /LEDs/LED_D37: track 111.8 -> 109.9 mm
- net COL6: track 205.8 -> 206.8 mm, vias 10 -> 9
- net COL4: track 212.3 -> 212.9 mm
- net ROW5: track 266.6 -> 266.1 mm, vias 20 -> 21
- net COL2: track 307.8 -> 307.6 mm, vias 12 -> 11
- net COL0: vias 19 -> 18
- net ROW1: vias 18 -> 20
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