File: unicorne-choc.kicad_pcb (KiCad board)
At the start: 2 copper layers, 299.9 x 118.8 mm, 173 parts, among them J1 Battery, J2 TPS43, J3 Expansion, J4 GPIO, J5 PAW3395 / PMW3360, J6 LED power in, Q1 AO3401A, Q2 2N7002, SW1 R0C0, SW10 R1C3, SW11 R1C4, SW12 R1C5, SW13 R2C0, SW14 R2C1, SW15 R2C2, SW16 R2C3, SW17 R2C4, SW18 R2C5, SW19 R0C6, SW2 R0C1, SW20 R1C6, SW21 R2C6, SW22 R3C0, SW23 R3C1, SW24 R3C2, SW25 R3C3, SW26 R3C4, SW27 R3C5, SW28 R4C0, SW29 R4C1, SW3 R0C2, SW30 R4C2, SW31 R4C3, SW32 R4C4, SW33 R4C5, SW34 R5C0, SW35 R5C1, SW36 R5C2, SW37 R5C3, SW38 R5C4, SW39 R5C5, SW4 R0C3, SW40 R3C6, SW41 R4C6, SW42 R5C6, SW43 Power, SW44 Reset, SW5 R0C4, SW6 R0C5, SW7 R1C0, SW8 R1C1, SW9 R1C2, U1 nice!nano v2, U2 SN74LV1T125

Commit message: Unrouted MX and Choc boards for hand routing
Both boards straight from gen_pcb.py (placement, outline, holes, silkscreen and
waves, no tracks, vias or zones).

Co-Authored-By: Claude Opus 5.5 <noreply@anthropic.com>
Parts:
- moved H4 1.68 mm to (78.0, 59.6)
- moved H5 0.79 mm to (224.7, 73.3)
- moved H1 0.56 mm to (133.5, 70.6)
- moved H8 0.25 mm to (283.0, 59.3)
- turned D1 to 74 degrees
- turned D10 to 74 degrees
- turned D11 to 74 degrees
- turned D12 to 74 degrees
- turned D13 to 74 degrees
- turned D14 to 74 degrees
- turned D15 to 74 degrees
- turned D16 to 74 degrees
- turned D17 to 74 degrees
- turned D18 to 74 degrees
- turned D19 to 74 degrees
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Routing:
- net GND: track 2002.2 -> 0.00 mm, vias 257 -> 0
- net LED_VDD: track 1026.4 -> 0.00 mm, vias 27 -> 0
- net COL0: track 397.0 -> 0.00 mm, vias 18 -> 0
- net /LEDs/LED_D51: track 353.5 -> 0.00 mm, vias 6 -> 0
- net COL1: track 348.8 -> 0.00 mm, vias 11 -> 0
- net COL2: track 307.6 -> 0.00 mm, vias 11 -> 0
- net ROW3: track 297.1 -> 0.00 mm, vias 22 -> 0
- net ROW0: track 273.8 -> 0.00 mm, vias 21 -> 0
- net COL3: track 268.8 -> 0.00 mm, vias 11 -> 0
- net ROW5: track 266.1 -> 0.00 mm, vias 21 -> 0
- net ROW1: track 263.9 -> 0.00 mm, vias 20 -> 0
- net ROW4: track 258.4 -> 0.00 mm, vias 22 -> 0
- net ROW2: track 256.9 -> 0.00 mm, vias 17 -> 0
- net COL4: track 212.9 -> 0.00 mm, vias 13 -> 0
- net COL6: track 206.8 -> 0.00 mm, vias 9 -> 0
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- removed copper zone on B.Cu, net GND
- removed copper zone on F.Cu, net GND

Commit message: Unrouted Choc board with the diode clear of the LED data lane
Co-Authored-By: Claude Opus 5.5 <noreply@anthropic.com>
Parts:
- moved D41 0.60 mm to (245.1, 120.6)
- moved D24 0.60 mm to (275.7, 50.9)
- moved D25 0.60 mm to (256.8, 53.8)
- moved D28 0.60 mm to (318.8, 63.2)
- moved D29 0.60 mm to (300.5, 68.5)
- moved D30 0.60 mm to (281.0, 69.1)
- moved D35 0.60 mm to (305.8, 86.7)
- moved D37 0.60 mm to (267.3, 90.3)
- moved D39 0.60 mm to (232.1, 105.4)
- moved D40 0.60 mm to (264.2, 114.1)
- moved D5 0.60 mm to (133.3, 64.9)
- moved D10 0.60 mm to (110.4, 75.7)
- moved D13 0.60 mm to (48.4, 85.1)
- moved D14 0.60 mm to (66.7, 90.3)
- moved D15 0.60 mm to (86.3, 91.0)
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