File: unicorne.kicad_pcb (KiCad board)
At the start: 2 copper layers, 0 parts

Commit message: Place MX and Choc PCBs from the layout and schematic
gen_pcb.py builds both boards: switches, diodes and LEDs from Corne v3
offsets, the nice!nano flush on the bottom, centre parts, outline,
36-key break lines with mouse bites, M2 holes, pad labels and a
nice!nano pin table on the silkscreen. Adds TPS43 / PAW3395-PMW3360
sensor pads and a 6x6 THT reset switch; underglow becomes SK6812MINI.

Co-Authored-By: Claude Opus 5.5 <noreply@anthropic.com>
Parts:
- added C1: 10uF, Capacitor_SMD:C_0805_2012Metric, B.Cu at (165.0, 82.2)
- added D1: 1N4148W, Diode_SMD:D_SOD-123, B.Cu at (61.1, 45.1)
- added D10: 1N4148W, Diode_SMD:D_SOD-123, B.Cu at (112.6, 72.2)
- added D11: 1N4148W, Diode_SMD:D_SOD-123, B.Cu at (130.2, 79.7)
- added D12: 1N4148W, Diode_SMD:D_SOD-123, B.Cu at (147.8, 87.3)
- added D13: 1N4148W, Diode_SMD:D_SOD-123, B.Cu at (50.6, 81.6)
- added D14: 1N4148W, Diode_SMD:D_SOD-123, B.Cu at (68.9, 86.9)
- added D15: 1N4148W, Diode_SMD:D_SOD-123, B.Cu at (88.4, 87.5)
- added D16: 1N4148W, Diode_SMD:D_SOD-123, B.Cu at (107.4, 90.5)
- added D17: 1N4148W, Diode_SMD:D_SOD-123, B.Cu at (125.0, 98.0)
- added D18: 1N4148W, Diode_SMD:D_SOD-123, B.Cu at (142.6, 105.5)
- added D19: 1N4148W, Diode_SMD:D_SOD-123, B.Cu at (110.4, 114.3)
- added D2: 1N4148W, Diode_SMD:D_SOD-123, B.Cu at (79.3, 50.3)
- added D20: 1N4148W, Diode_SMD:D_SOD-123, B.Cu at (129.1, 124.5)
- added D21: 1N4148W, Diode_SMD:D_SOD-123, B.Cu at (148.4, 125.0)
- added D22: 1N4148W, Diode_SMD:D_SOD-123, B.Cu at (313.6, 40.9)
- added D23: 1N4148W, Diode_SMD:D_SOD-123, B.Cu at (295.3, 46.1)
- added D24: 1N4148W, Diode_SMD:D_SOD-123, B.Cu at (275.7, 46.8)
- added D25: 1N4148W, Diode_SMD:D_SOD-123, B.Cu at (256.8, 49.8)
- added D26: 1N4148W, Diode_SMD:D_SOD-123, B.Cu at (239.2, 57.3)
- added D27: 1N4148W, Diode_SMD:D_SOD-123, B.Cu at (221.6, 64.8)
- added D28: 1N4148W, Diode_SMD:D_SOD-123, B.Cu at (318.8, 59.2)
- added D29: 1N4148W, Diode_SMD:D_SOD-123, B.Cu at (300.6, 64.4)
- added D3: 1N4148W, Diode_SMD:D_SOD-123, B.Cu at (98.9, 51.0)
- added D30: 1N4148W, Diode_SMD:D_SOD-123, B.Cu at (281.0, 65.1)
- added D31: 1N4148W, Diode_SMD:D_SOD-123, B.Cu at (262.1, 68.0)
- added D32: 1N4148W, Diode_SMD:D_SOD-123, B.Cu at (244.5, 75.5)
- added D33: 1N4148W, Diode_SMD:D_SOD-123, B.Cu at (226.8, 83.1)
- added D34: 1N4148W, Diode_SMD:D_SOD-123, B.Cu at (324.1, 77.4)
- added D35: 1N4148W, Diode_SMD:D_SOD-123, B.Cu at (305.8, 82.7)
- added D36: 1N4148W, Diode_SMD:D_SOD-123, B.Cu at (286.2, 83.3)
- added D37: 1N4148W, Diode_SMD:D_SOD-123, B.Cu at (267.3, 86.3)
- added D38: 1N4148W, Diode_SMD:D_SOD-123, B.Cu at (249.7, 93.8)
- added D39: 1N4148W, Diode_SMD:D_SOD-123, B.Cu at (232.1, 101.3)
- added D4: 1N4148W, Diode_SMD:D_SOD-123, B.Cu at (117.8, 54.0)
- added D40: 1N4148W, Diode_SMD:D_SOD-123, B.Cu at (264.2, 110.1)
- added D41: 1N4148W, Diode_SMD:D_SOD-123, B.Cu at (244.0, 116.7)
- added D42: 1N4148W, Diode_SMD:D_SOD-123, B.Cu at (222.6, 135.6)
- added D5: 1N4148W, Diode_SMD:D_SOD-123, B.Cu at (135.4, 61.5)
- added D6: 1N4148W, Diode_SMD:D_SOD-123, B.Cu at (153.1, 69.0)
- added D7: 1N4148W, Diode_SMD:D_SOD-123, B.Cu at (55.8, 63.4)
- added D8: 1N4148W, Diode_SMD:D_SOD-123, B.Cu at (74.1, 68.6)
- added D9: 1N4148W, Diode_SMD:D_SOD-123, B.Cu at (93.7, 69.3)
- added H1: M2, MountingHole:MountingHole_2.2mm_M2_ISO7380, F.Cu at (134.3, 72.3)
- added H10: M2, MountingHole:MountingHole_2.2mm_M2_ISO7380, F.Cu at (194.0, 133.6)
- added H2: M2, MountingHole:MountingHole_2.2mm_M2_ISO7380, F.Cu at (97.0, 101.5)
- added H3: M2, MountingHole:MountingHole_2.2mm_M2_ISO7380, F.Cu at (134.4, 121.6)
- added H4: M2, MountingHole:MountingHole_2.2mm_M2_ISO7380, F.Cu at (78.0, 59.8)
- added H5: M2, MountingHole:MountingHole_2.2mm_M2_ISO7380, F.Cu at (225.7, 72.3)
- added H6: M2, MountingHole:MountingHole_2.2mm_M2_ISO7380, F.Cu at (269.7, 95.2)
- added H7: M2, MountingHole:MountingHole_2.2mm_M2_ISO7380, F.Cu at (225.6, 121.6)
- added H8: M2, MountingHole:MountingHole_2.2mm_M2_ISO7380, F.Cu at (282.0, 59.8)
- added H9: M2, MountingHole:MountingHole_2.2mm_M2_ISO7380, F.Cu at (166.0, 133.6)
- added J1: Battery, Connector_Wire:SolderWire-0.5sqmm_1x02_P4.8mm_D0.9mm_OD2.3mm, F.Cu at (177.6, 133.6)
- added J2: TPS43, Connector_PinHeader_2.54mm:PinHeader_1x06_P2.54mm_Vertical, F.Cu at (186.3, 125.1)
- added J3: Expansion, Connector_PinHeader_2.54mm:PinHeader_1x06_P2.54mm_Vertical, B.Cu at (193.5, 67.8)
- added J4: GPIO, Connector_PinHeader_2.54mm:PinHeader_1x04_P2.54mm_Vertical, B.Cu at (166.5, 61.8)
- added J5: PAW3395 / PMW3360, Connector_PinHeader_2.54mm:PinHeader_1x08_P2.54mm_Vertical, F.Cu at (171.1, 120.1)
- added JP1: LED data, Jumper:SolderJumper-2_P1.3mm_Open_RoundedPad1.0x1.5mm, B.Cu at (198.0, 77.7)
- added LED1: SK6812MINI, LED_SMD:LED_SK6812MINI_PLCC4_3.5x3.5mm_P1.75mm, B.Cu at (69.5, 57.1)
- added LED10: SK6812MINI, LED_SMD:LED_SK6812MINI_PLCC4_3.5x3.5mm_P1.75mm, B.Cu at (295.8, 75.3)
- added LED11: SK6812MINI, LED_SMD:LED_SK6812MINI_PLCC4_3.5x3.5mm_P1.75mm, B.Cu at (262.5, 97.2)
- added LED12: SK6812MINI, LED_SMD:LED_SK6812MINI_PLCC4_3.5x3.5mm_P1.75mm, B.Cu at (227.3, 112.3)
- added LED13: SK6812MINI-E, LED_SMD:LED_SK6812MINI-E_3.2x2.8mm_P1.5mm_ReverseMount, B.Cu at (70.7, 52.8)
- added LED14: SK6812MINI-E, LED_SMD:LED_SK6812MINI-E_3.2x2.8mm_P1.5mm_ReverseMount, B.Cu at (90.3, 53.5)
- added LED15: SK6812MINI-E, LED_SMD:LED_SK6812MINI-E_3.2x2.8mm_P1.5mm_ReverseMount, B.Cu at (109.2, 56.4)
- added LED16: SK6812MINI-E, LED_SMD:LED_SK6812MINI-E_3.2x2.8mm_P1.5mm_ReverseMount, B.Cu at (126.8, 63.9)
- added LED17: SK6812MINI-E, LED_SMD:LED_SK6812MINI-E_3.2x2.8mm_P1.5mm_ReverseMount, B.Cu at (144.4, 71.5)
- added LED18: SK6812MINI-E, LED_SMD:LED_SK6812MINI-E_3.2x2.8mm_P1.5mm_ReverseMount, B.Cu at (139.2, 89.7)
- added LED19: SK6812MINI-E, LED_SMD:LED_SK6812MINI-E_3.2x2.8mm_P1.5mm_ReverseMount, B.Cu at (121.6, 82.2)
- added LED2: SK6812MINI, LED_SMD:LED_SK6812MINI_PLCC4_3.5x3.5mm_P1.75mm, B.Cu at (108.0, 60.7)
- added LED20: SK6812MINI-E, LED_SMD:LED_SK6812MINI-E_3.2x2.8mm_P1.5mm_ReverseMount, B.Cu at (104.0, 74.7)
- added LED21: SK6812MINI-E, LED_SMD:LED_SK6812MINI-E_3.2x2.8mm_P1.5mm_ReverseMount, B.Cu at (85.0, 71.7)
- added LED22: SK6812MINI-E, LED_SMD:LED_SK6812MINI-E_3.2x2.8mm_P1.5mm_ReverseMount, B.Cu at (65.5, 71.1)
- added LED23: SK6812MINI-E, LED_SMD:LED_SK6812MINI-E_3.2x2.8mm_P1.5mm_ReverseMount, B.Cu at (60.2, 89.3)
- added LED24: SK6812MINI-E, LED_SMD:LED_SK6812MINI-E_3.2x2.8mm_P1.5mm_ReverseMount, B.Cu at (79.8, 90.0)
- added LED25: SK6812MINI-E, LED_SMD:LED_SK6812MINI-E_3.2x2.8mm_P1.5mm_ReverseMount, B.Cu at (98.7, 93.0)
- added LED26: SK6812MINI-E, LED_SMD:LED_SK6812MINI-E_3.2x2.8mm_P1.5mm_ReverseMount, B.Cu at (116.3, 100.5)
- added LED27: SK6812MINI-E, LED_SMD:LED_SK6812MINI-E_3.2x2.8mm_P1.5mm_ReverseMount, B.Cu at (133.9, 108.0)
- added LED28: SK6812MINI-E, LED_SMD:LED_SK6812MINI-E_3.2x2.8mm_P1.5mm_ReverseMount, B.Cu at (101.8, 116.7)
- added LED29: SK6812MINI-E, LED_SMD:LED_SK6812MINI-E_3.2x2.8mm_P1.5mm_ReverseMount, B.Cu at (120.1, 124.7)
- added LED3: SK6812MINI, LED_SMD:LED_SK6812MINI_PLCC4_3.5x3.5mm_P1.75mm, B.Cu at (143.2, 75.7)
- added LED30: SK6812MINI-E, LED_SMD:LED_SK6812MINI-E_3.2x2.8mm_P1.5mm_ReverseMount, B.Cu at (146.2, 133.7)
- added LED31: SK6812MINI-E, LED_SMD:LED_SK6812MINI-E_3.2x2.8mm_P1.5mm_ReverseMount, B.Cu at (289.3, 52.8)
- added LED32: SK6812MINI-E, LED_SMD:LED_SK6812MINI-E_3.2x2.8mm_P1.5mm_ReverseMount, B.Cu at (269.7, 53.5)
- added LED33: SK6812MINI-E, LED_SMD:LED_SK6812MINI-E_3.2x2.8mm_P1.5mm_ReverseMount, B.Cu at (250.8, 56.4)
- added LED34: SK6812MINI-E, LED_SMD:LED_SK6812MINI-E_3.2x2.8mm_P1.5mm_ReverseMount, B.Cu at (233.2, 63.9)
- added LED35: SK6812MINI-E, LED_SMD:LED_SK6812MINI-E_3.2x2.8mm_P1.5mm_ReverseMount, B.Cu at (215.6, 71.5)
- added LED36: SK6812MINI-E, LED_SMD:LED_SK6812MINI-E_3.2x2.8mm_P1.5mm_ReverseMount, B.Cu at (220.8, 89.7)
- added LED37: SK6812MINI-E, LED_SMD:LED_SK6812MINI-E_3.2x2.8mm_P1.5mm_ReverseMount, B.Cu at (238.4, 82.2)
- added LED38: SK6812MINI-E, LED_SMD:LED_SK6812MINI-E_3.2x2.8mm_P1.5mm_ReverseMount, B.Cu at (256.0, 74.7)
- added LED39: SK6812MINI-E, LED_SMD:LED_SK6812MINI-E_3.2x2.8mm_P1.5mm_ReverseMount, B.Cu at (275.0, 71.7)
- added LED4: SK6812MINI, LED_SMD:LED_SK6812MINI_PLCC4_3.5x3.5mm_P1.75mm, B.Cu at (64.2, 75.3)
- added LED40: SK6812MINI-E, LED_SMD:LED_SK6812MINI-E_3.2x2.8mm_P1.5mm_ReverseMount, B.Cu at (294.5, 71.1)
- added LED41: SK6812MINI-E, LED_SMD:LED_SK6812MINI-E_3.2x2.8mm_P1.5mm_ReverseMount, B.Cu at (299.8, 89.3)
- added LED42: SK6812MINI-E, LED_SMD:LED_SK6812MINI-E_3.2x2.8mm_P1.5mm_ReverseMount, B.Cu at (280.2, 90.0)
- added LED43: SK6812MINI-E, LED_SMD:LED_SK6812MINI-E_3.2x2.8mm_P1.5mm_ReverseMount, B.Cu at (261.3, 93.0)
- added LED44: SK6812MINI-E, LED_SMD:LED_SK6812MINI-E_3.2x2.8mm_P1.5mm_ReverseMount, B.Cu at (243.7, 100.5)
- added LED45: SK6812MINI-E, LED_SMD:LED_SK6812MINI-E_3.2x2.8mm_P1.5mm_ReverseMount, B.Cu at (226.1, 108.0)
- added LED46: SK6812MINI-E, LED_SMD:LED_SK6812MINI-E_3.2x2.8mm_P1.5mm_ReverseMount, B.Cu at (258.2, 116.7)
- added LED47: SK6812MINI-E, LED_SMD:LED_SK6812MINI-E_3.2x2.8mm_P1.5mm_ReverseMount, B.Cu at (239.9, 124.7)
- added LED48: SK6812MINI-E, LED_SMD:LED_SK6812MINI-E_3.2x2.8mm_P1.5mm_ReverseMount, B.Cu at (213.8, 133.7)
- added LED49: SK6812MINI-E, LED_SMD:LED_SK6812MINI-E_3.2x2.8mm_P1.5mm_ReverseMount, B.Cu at (52.4, 47.6)
- added LED5: SK6812MINI, LED_SMD:LED_SK6812MINI_PLCC4_3.5x3.5mm_P1.75mm, B.Cu at (97.5, 97.2)
- added LED50: SK6812MINI-E, LED_SMD:LED_SK6812MINI-E_3.2x2.8mm_P1.5mm_ReverseMount, B.Cu at (47.2, 65.8)
- added LED51: SK6812MINI-E, LED_SMD:LED_SK6812MINI-E_3.2x2.8mm_P1.5mm_ReverseMount, B.Cu at (42.0, 84.1)
- added LED52: SK6812MINI-E, LED_SMD:LED_SK6812MINI-E_3.2x2.8mm_P1.5mm_ReverseMount, B.Cu at (307.6, 47.6)
- added LED53: SK6812MINI-E, LED_SMD:LED_SK6812MINI-E_3.2x2.8mm_P1.5mm_ReverseMount, B.Cu at (312.8, 65.8)
- added LED54: SK6812MINI-E, LED_SMD:LED_SK6812MINI-E_3.2x2.8mm_P1.5mm_ReverseMount, B.Cu at (318.0, 84.1)
- added LED6: SK6812MINI, LED_SMD:LED_SK6812MINI_PLCC4_3.5x3.5mm_P1.75mm, B.Cu at (132.7, 112.3)
- added LED7: SK6812MINI, LED_SMD:LED_SK6812MINI_PLCC4_3.5x3.5mm_P1.75mm, B.Cu at (290.5, 57.1)
- added LED8: SK6812MINI, LED_SMD:LED_SK6812MINI_PLCC4_3.5x3.5mm_P1.75mm, B.Cu at (252.0, 60.7)
- added LED9: SK6812MINI, LED_SMD:LED_SK6812MINI_PLCC4_3.5x3.5mm_P1.75mm, B.Cu at (216.8, 75.7)
- added MB1, MB2: mouse bites, , F.Cu at (0.00, 0.00)
- added Q1: AO3401A, Package_TO_SOT_SMD:SOT-23, B.Cu at (165.0, 73.7)
- added Q2: 2N7002, Package_TO_SOT_SMD:SOT-23, B.Cu at (165.0, 78.2)
- added R1: 100k, Resistor_SMD:R_0603_1608Metric, B.Cu at (168.5, 73.7)
- added R2: 100k, Resistor_SMD:R_0603_1608Metric, B.Cu at (168.5, 78.2)
- added R3: 4.7k, Resistor_SMD:R_0603_1608Metric, B.Cu at (177.0, 129.1)
- added R4: 4.7k, Resistor_SMD:R_0603_1608Metric, B.Cu at (180.0, 129.1)
- added R5: 10k, Resistor_SMD:R_0603_1608Metric, B.Cu at (183.0, 129.1)
- added SW1: R0C0, unicorne:SW_Hotswap_Kailh_MX_1.00u, F.Cu at (53.8, 43.0)
- added SW10: R1C3, unicorne:SW_Hotswap_Kailh_MX_1.00u, F.Cu at (105.3, 70.1)
- added SW11: R1C4, unicorne:SW_Hotswap_Kailh_MX_1.00u, F.Cu at (122.9, 77.6)
- added SW12: R1C5, unicorne:SW_Hotswap_Kailh_MX_1.00u, F.Cu at (140.5, 85.2)
- added SW13: R2C0, unicorne:SW_Hotswap_Kailh_MX_1.00u, F.Cu at (43.3, 79.5)
- added SW14: R2C1, unicorne:SW_Hotswap_Kailh_MX_1.00u, F.Cu at (61.5, 84.8)
- added SW15: R2C2, unicorne:SW_Hotswap_Kailh_MX_1.00u, F.Cu at (81.1, 85.4)
- added SW16: R2C3, unicorne:SW_Hotswap_Kailh_MX_1.00u, F.Cu at (100.0, 88.4)
- added SW17: R2C4, unicorne:SW_Hotswap_Kailh_MX_1.00u, F.Cu at (117.6, 95.9)
- added SW18: R2C5, unicorne:SW_Hotswap_Kailh_MX_1.00u, F.Cu at (135.2, 103.4)
- added SW19: R0C6, unicorne:SW_Hotswap_Kailh_MX_1.00u, F.Cu at (103.1, 112.2)
- added SW2: R0C1, unicorne:SW_Hotswap_Kailh_MX_1.00u, F.Cu at (72.0, 48.2)
- added SW20: R1C6, unicorne:SW_Hotswap_Kailh_MX_1.00u, F.Cu at (122.5, 120.6)
- added SW21: R2C6, unicorne:SW_Hotswap_Kailh_MX_1.50u, F.Cu at (142.9, 130.3)
- added SW22: R3C0, unicorne:SW_Hotswap_Kailh_MX_1.00u, F.Cu at (306.2, 43.0)
- added SW23: R3C1, unicorne:SW_Hotswap_Kailh_MX_1.00u, F.Cu at (288.0, 48.2)
- added SW24: R3C2, unicorne:SW_Hotswap_Kailh_MX_1.00u, F.Cu at (268.4, 48.9)
- added SW25: R3C3, unicorne:SW_Hotswap_Kailh_MX_1.00u, F.Cu at (249.5, 51.9)
- added SW26: R3C4, unicorne:SW_Hotswap_Kailh_MX_1.00u, F.Cu at (231.9, 59.4)
- added SW27: R3C5, unicorne:SW_Hotswap_Kailh_MX_1.00u, F.Cu at (214.3, 66.9)
- added SW28: R4C0, unicorne:SW_Hotswap_Kailh_MX_1.00u, F.Cu at (311.5, 61.3)
- added SW29: R4C1, unicorne:SW_Hotswap_Kailh_MX_1.00u, F.Cu at (293.2, 66.5)
- added SW3: R0C2, unicorne:SW_Hotswap_Kailh_MX_1.00u, F.Cu at (91.6, 48.9)
- added SW30: R4C2, unicorne:SW_Hotswap_Kailh_MX_1.00u, F.Cu at (273.6, 67.2)
- added SW31: R4C3, unicorne:SW_Hotswap_Kailh_MX_1.00u, F.Cu at (254.7, 70.1)
- added SW32: R4C4, unicorne:SW_Hotswap_Kailh_MX_1.00u, F.Cu at (237.1, 77.6)
- added SW33: R4C5, unicorne:SW_Hotswap_Kailh_MX_1.00u, F.Cu at (219.5, 85.2)
- added SW34: R5C0, unicorne:SW_Hotswap_Kailh_MX_1.00u, F.Cu at (316.7, 79.5)
- added SW35: R5C1, unicorne:SW_Hotswap_Kailh_MX_1.00u, F.Cu at (298.5, 84.8)
- added SW36: R5C2, unicorne:SW_Hotswap_Kailh_MX_1.00u, F.Cu at (278.9, 85.4)
- added SW37: R5C3, unicorne:SW_Hotswap_Kailh_MX_1.00u, F.Cu at (260.0, 88.4)
- added SW38: R5C4, unicorne:SW_Hotswap_Kailh_MX_1.00u, F.Cu at (242.4, 95.9)
- added SW39: R5C5, unicorne:SW_Hotswap_Kailh_MX_1.00u, F.Cu at (224.8, 103.4)
- added SW4: R0C3, unicorne:SW_Hotswap_Kailh_MX_1.00u, F.Cu at (110.5, 51.9)
- added SW40: R3C6, unicorne:SW_Hotswap_Kailh_MX_1.00u, F.Cu at (256.9, 112.2)
- added SW41: R4C6, unicorne:SW_Hotswap_Kailh_MX_1.00u, F.Cu at (237.5, 120.6)
- added SW42: R5C6, unicorne:SW_Hotswap_Kailh_MX_1.50u, F.Cu at (217.1, 130.3)
- added SW43: Power, Button_Switch_SMD:SW_SPDT_Shouhan_MSK12C02, B.Cu at (165.0, 55.7)
- added SW44: Reset, Button_Switch_THT:SW_PUSH_6mm_H5mm, B.Cu at (192.2, 61.4)
- added SW5: R0C4, unicorne:SW_Hotswap_Kailh_MX_1.00u, F.Cu at (128.1, 59.4)
- added SW6: R0C5, unicorne:SW_Hotswap_Kailh_MX_1.00u, F.Cu at (145.7, 66.9)
- added SW7: R1C0, unicorne:SW_Hotswap_Kailh_MX_1.00u, F.Cu at (48.5, 61.3)
- added SW8: R1C1, unicorne:SW_Hotswap_Kailh_MX_1.00u, F.Cu at (66.8, 66.5)
- added SW9: R1C2, unicorne:SW_Hotswap_Kailh_MX_1.00u, F.Cu at (86.3, 67.2)
- added U1: nice!nano v2, unicorne:nice_nano, B.Cu at (180.0, 71.4)
Other:
- board outline added: 299.9 x 118.8 mm
- board text added: "0.11"
- board text added: "0.24"
- board text added: "1.00"
- board text added: "3V3"
- board text added: "3V3 out"
- board text added: "B+"
- board text added: "B-"
- board text added: "BATT"
- board text added: "COL0"
- board text added: "COL1"
- board text added: "COL2"
- board text added: "COL3"
- board text added: "COL4"
- board text added: "COL5"
- board text added: "COL6"
- board text added: "CS"
- board text added: "GND"
- board text added: "GPIO"
- board text added: "GPIO / sens CS"
- board text added: "GPIO / sens MISO"
- board text added: "LED power on"
- board text added: "MISO"
- board text added: "MOSI"
- board text added: "MOT"
- board text added: "P0.02"
- board text added: "P0.06"
- board text added: "P0.08"
- board text added: "P0.09"
- board text added: "P0.10"
- board text added: "P0.11"
- board text added: "P0.17"
- board text added: "P0.20"
- board text added: "P0.22"
- board text added: "P0.24"
- board text added: "P0.29"
- board text added: "P0.31"
- board text added: "P1.00"
- board text added: "P1.01"
- board text added: "P1.02"
- board text added: "P1.04"
- board text added: "P1.06"
- board text added: "P1.07"
- board text added: "P1.11"
- board text added: "P1.13"
- board text added: "P1.15"
- board text added: "RAW"
- board text added: "RDY"
- board text added: "ROW0"
- board text added: "ROW1"
- board text added: "ROW2"
- board text added: "ROW3"
- board text added: "ROW4"
- board text added: "ROW5"
- board text added: "RST"
- board text added: "RX"
- board text added: "SCK"
- board text added: "SCL"
- board text added: "SCL / sens SCK"
- board text added: "SDA"
- board text added: "SDA / sens MOSI"
- board text added: "SENSOR"
- board text added: "TP RDY / sens MOT"
- board text added: "TPS43"
- board text added: "TX"
- board text added: "TX / LED data"
- board text added: "UART/I2C"
- board text added: "VCC"
- board text added: "battery (switch)"
- board text added: "nice!nano pins"
- board text added: "reset button"

Commit message: Rework LED power, break lines and centre placement; add routing tools
- LED supply chosen by solder jumper JP2: nice!nano VCC, or an external
  supply on new LED IN pads (J6); never the battery pin. SN74LV1T125
  level shifter (U2) with bypass jumper JP3.
- Centre parts rearranged so the nice!nano's matrix pins are clear.
- 0805 hand-solder passives; LED chain runs left to right per row.
- Break lines: no sliver slots, perforated end to end, tabs over the lanes.
- Mounting holes stay inside the board and off the routing lanes.
- Routing tools (lanes, Freerouting driver, maze router) and placeholder
  STEP models. Boards are committed placed but unrouted.

Co-Authored-By: Claude Opus 5.5 <noreply@anthropic.com>
Parts:
- added C2: 100nF, Capacitor_SMD:C_0805_2012Metric_Pad1.18x1.45mm_HandSolder, B.Cu at (201.5, 59.2)
- added J6: LED power in, Connector_PinHeader_2.54mm:PinHeader_1x02_P2.54mm_Vertical, F.Cu at (188.0, 132.3)
- added JP2: LED source, Jumper:SolderJumper-3_P1.3mm_Open_RoundedPad1.0x1.5mm, B.Cu at (202.1, 75.7)
- added JP3: U2 bypass, Jumper:SolderJumper-2_P1.3mm_Open_RoundedPad1.0x1.5mm, B.Cu at (202.0, 68.2)
- added U2: SN74LV1T125, Package_TO_SOT_SMD:SOT-23-5_HandSoldering, B.Cu at (201.5, 63.6)
- C1: footprint Capacitor_SMD:C_0805_2012Metric -> Capacitor_SMD:C_0805_2012Metric_Pad1.18x1.45mm_HandSolder
- R1, R2, R3, R4, R5: footprint Resistor_SMD:R_0603_1608Metric -> Resistor_SMD:R_0805_2012Metric_Pad1.20x1.40mm_HandSolder
- moved LED31 76.0 mm to (215.6, 71.5)
- moved LED35 76.0 mm to (289.3, 52.8)
- moved LED18 76.0 mm to (65.5, 71.1)
- moved LED22 76.0 mm to (139.2, 89.7)
- moved LED41 76.0 mm to (226.1, 108.0)
- moved LED45 76.0 mm to (299.8, 89.3)
- moved LED32 38.0 mm to (233.2, 63.9)
- moved LED34 38.0 mm to (269.7, 53.5)
- moved LED42 38.0 mm to (243.7, 100.5)
- moved LED44 38.0 mm to (280.2, 90.0)
- moved LED19 38.0 mm to (85.0, 71.7)
- moved LED21 38.0 mm to (121.6, 82.2)
- moved Q2 34.6 mm to (198.0, 67.7)
- moved Q1 33.1 mm to (198.0, 75.7)
- moved C1 33.0 mm to (198.0, 83.7)
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Connections:
- JP1 pad 2: LED_DIN -> /LED_DATA
- Q1 pad 2: /VBAT -> /LED_SRC
- R1 pad 1: /VBAT -> /LED_SRC
Other:
- outline, holes or cut-outs redrawn
- board text added: "EXT"
- board text added: "LED IN"
- board text added: "V+"

Commit message: Route the MX board
finish_route.py lays fixed lanes on the key grid (columns on top; rows,
LED data and LED supply on the bottom), then routes KiCad's remaining
ratsnest with the maze router, pours GND on both layers and stitches
them. DRC: 0 unconnected, 0 copper violations, matches the schematic.

LED chain reordered to cross the board once; Q1 rotated so its source
faces JP2.

Co-Authored-By: Claude Opus 5.5 <noreply@anthropic.com>
Parts:
- LED10, LED11, LED12, LED7, LED8, LED9: value SK6812MINI -> SK6812MINI-E; footprint LED_SMD:LED_SK6812MINI_PLCC4_3.5x3.5mm_P1.75mm -> LED_SMD:LED_SK6812MINI-E_3.2x2.8mm_P1.5mm_ReverseMount
- LED43, LED44, LED45, LED46, LED47, LED48: value SK6812MINI-E -> SK6812MINI; footprint LED_SMD:LED_SK6812MINI-E_3.2x2.8mm_P1.5mm_ReverseMount -> LED_SMD:LED_SK6812MINI_PLCC4_3.5x3.5mm_P1.75mm
- moved LED51 276.1 mm to (318.0, 84.1), turned to 16 degrees
- moved LED54 276.1 mm to (42.0, 84.1), turned to -16 degrees
- moved LED50 265.6 mm to (312.8, 65.8), turned to 16 degrees
- moved LED53 265.6 mm to (47.2, 65.8), turned to -16 degrees
- moved LED49 255.1 mm to (307.6, 47.6), turned to 16 degrees
- moved LED52 255.1 mm to (52.4, 47.6), turned to -16 degrees
- moved LED7 219.9 mm to (70.7, 52.8), turned to -16 degrees
- moved LED10 169.3 mm to (126.8, 63.9), turned to -16 degrees
- moved LED12 167.0 mm to (65.5, 71.1), turned to -16 degrees
- moved LED8 161.9 mm to (90.3, 53.5), turned to -16 degrees
- moved LED30 130.1 mm to (250.8, 56.4), turned to 16 degrees
- moved LED29 128.4 mm to (233.2, 63.9), turned to 16 degrees
- moved LED26 125.9 mm to (239.9, 124.7), turned to 31 degrees
- moved LED27 124.6 mm to (258.2, 116.7), turned to 16 degrees
- moved LED28 122.5 mm to (215.6, 71.5), turned to 16 degrees
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Connections:
- LED10 pad 1: /LEDs/LED_D10 -> GND
- LED10 pad 2: GND -> /LEDs/LED_D9
- LED10 pad 3: /LEDs/LED_D9 -> LED_VDD
- LED10 pad 4: LED_VDD -> /LEDs/LED_D10
- LED11 pad 1: /LEDs/LED_D11 -> GND
- LED11 pad 2: GND -> /LEDs/LED_D10
- LED11 pad 3: /LEDs/LED_D10 -> LED_VDD
- LED11 pad 4: LED_VDD -> /LEDs/LED_D11
- LED12 pad 1: /LEDs/LED_D12 -> GND
- LED12 pad 2: GND -> /LEDs/LED_D11
- LED12 pad 3: /LEDs/LED_D11 -> LED_VDD
- LED12 pad 4: LED_VDD -> /LEDs/LED_D12
- LED43 pad 1: GND -> /LEDs/LED_D43
- LED43 pad 2: /LEDs/LED_D42 -> GND
- LED43 pad 3: LED_VDD -> /LEDs/LED_D42
- LED43 pad 4: /LEDs/LED_D43 -> LED_VDD
- LED44 pad 1: GND -> /LEDs/LED_D44
- LED44 pad 2: /LEDs/LED_D43 -> GND
- LED44 pad 3: LED_VDD -> /LEDs/LED_D43
- LED44 pad 4: /LEDs/LED_D44 -> LED_VDD
- LED45 pad 1: GND -> /LEDs/LED_D45
- LED45 pad 2: /LEDs/LED_D44 -> GND
- LED45 pad 3: LED_VDD -> /LEDs/LED_D44
- LED45 pad 4: /LEDs/LED_D45 -> LED_VDD
- LED46 pad 1: GND -> /LEDs/LED_D46
- LED46 pad 2: /LEDs/LED_D45 -> GND
- LED46 pad 3: LED_VDD -> /LEDs/LED_D45
- LED46 pad 4: /LEDs/LED_D46 -> LED_VDD
- LED47 pad 1: GND -> /LEDs/LED_D47
- LED47 pad 2: /LEDs/LED_D46 -> GND
- LED47 pad 3: LED_VDD -> /LEDs/LED_D46
- LED47 pad 4: /LEDs/LED_D47 -> LED_VDD
- LED48 pad 1: GND -> /LEDs/LED_D48
- LED48 pad 2: /LEDs/LED_D47 -> GND
- LED48 pad 3: LED_VDD -> /LEDs/LED_D47
- LED48 pad 4: /LEDs/LED_D48 -> LED_VDD
- LED7 pad 1: /LEDs/LED_D7 -> GND
- LED7 pad 2: GND -> /LEDs/LED_D6
- LED7 pad 3: /LEDs/LED_D6 -> LED_VDD
- LED7 pad 4: LED_VDD -> /LEDs/LED_D7
- LED8 pad 1: /LEDs/LED_D8 -> GND
- LED8 pad 2: GND -> /LEDs/LED_D7
- LED8 pad 3: /LEDs/LED_D7 -> LED_VDD
- LED8 pad 4: LED_VDD -> /LEDs/LED_D8
- LED9 pad 1: /LEDs/LED_D9 -> GND
- LED9 pad 2: GND -> /LEDs/LED_D8
- LED9 pad 3: /LEDs/LED_D8 -> LED_VDD
- LED9 pad 4: LED_VDD -> /LEDs/LED_D9
Routing:
- net GND: track 0.00 -> 1724.2 mm, vias 0 -> 233
- net LED_VDD: track 0.00 -> 1100.3 mm, vias 0 -> 27
- net COL0: track 0.00 -> 398.4 mm, vias 0 -> 14
- net COL1: track 0.00 -> 337.6 mm, vias 0 -> 9
- net /LEDs/LED_D51: track 0.00 -> 325.0 mm, vias 0 -> 14
- net COL2: track 0.00 -> 299.8 mm, vias 0 -> 6
- net COL3: track 0.00 -> 266.1 mm, vias 0 -> 9
- net COL4: track 0.00 -> 218.0 mm, vias 0 -> 11
- net COL6: track 0.00 -> 217.0 mm, vias 0 -> 9
- net ROW3: track 0.00 -> 211.7 mm, vias 0 -> 6
- net ROW5: track 0.00 -> 205.7 mm, vias 0 -> 3
- net ROW4: track 0.00 -> 188.0 mm, vias 0 -> 2
- net ROW0: track 0.00 -> 186.7 mm, vias 0 -> 2
- net ROW1: track 0.00 -> 183.9 mm, vias 0 -> 2
- net COL5: track 0.00 -> 182.4 mm, vias 0 -> 7
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- added copper zone on B.Cu, net GND
- added copper zone on F.Cu, net GND

Commit message: Route the Choc board
lanes.py now has per-switch-type lane layouts. Choc: rows run above the
sockets (y -8.0), reached from each cathode by a short top-layer hop
between the switch holes; LED data and supply below the diode; where the
next column sits lower the row lane jogs on the top layer. Break-line
tabs and mounting-hole keep-outs follow the lanes, and finish_route.py
nudges any hole the lanes still touch and retries failed connections
first. MX routing is unchanged.

DRC (Choc): 0 unconnected, 0 copper violations.

Co-Authored-By: Claude Opus 5.5 <noreply@anthropic.com>
Routing:
- net GND: track 1724.2 -> 1685.8 mm, vias 233 -> 231
- net /LEDs/LED_D52: track 33.3 -> 29.2 mm
- net COL0: track 398.4 -> 402.0 mm
- net /LEDs/LED_D4: track 55.8 -> 52.3 mm, vias 2 -> 4
- net /LEDs/LED_D6: track 5.49 -> 7.31 mm
- net COL2: track 299.8 -> 297.9 mm, vias 6 -> 7
- net /LEDs/LED_D47: track 36.5 -> 34.7 mm
- net /LEDs/LED_D11: track 97.9 -> 99.0 mm
- net /LEDs/LED_D51: track 325.0 -> 326.0 mm
- net LED_VDD: track 1100.3 -> 1100.9 mm, vias 27 -> 34
- net /LEDs/LED_D43: track 48.5 -> 47.9 mm

Commit message: Add 3D models and STEP export
Project footprints point at models in lib/3d/: Kailh MX and Choc hotswap
sockets and the Choc V1 switch (keyswitch-kicad-library), plus placeholder
boxes for the nice!nano, TPS43, MX switch, SK6812MINI and MSK-12C02 (the
last two copied from the stock library with a model added). The trackpad
model sits on a board-only footprint; bare pads carry no model.
export_3d.py writes export/unicorne-{mx,choc}.step; renders alongside.

Both boards regenerated and re-routed: DRC 0 unconnected, 0 copper
violations.

Co-Authored-By: Claude Opus 5.5 <noreply@anthropic.com>
Parts:
- added TP1: TPS43, , F.Cu at (180.0, 101.1)
- LED1, LED2, LED3, LED4, LED43, LED44, LED45, LED46, LED47, LED48, LED5, LED6: footprint LED_SMD:LED_SK6812MINI_PLCC4_3.5x3.5mm_P1.75mm -> unicorne:LED_SK6812MINI_PLCC4_3.5x3.5mm_P1.75mm
- SW43: footprint Button_Switch_SMD:SW_SPDT_Shouhan_MSK12C02 -> unicorne:SW_SPDT_Shouhan_MSK12C02
Routing:
- net GND: track 1685.8 -> 1710.6 mm, vias 231 -> 227
- net LED_VDD: track 1100.9 -> 1093.8 mm, vias 34 -> 30
- net /LEDs/LED_D52: track 29.2 -> 33.3 mm
- net COL0: track 402.0 -> 398.4 mm
- net COL2: track 297.9 -> 299.8 mm, vias 7 -> 6
- net ROW5: track 205.7 -> 206.3 mm
