File: unicorne.kicad_pcb (KiCad board)
At the start: 2 copper layers, 293.4 x 118.8 mm, 172 parts, among them J1 Battery, J2 TPS43, J3 Expansion, J4 GPIO, J5 PAW3395 / PMW3360, J6 LED power in, Q1 AO3401A, Q2 2N7002, SW1 R0C0, SW10 R1C3, SW11 R1C4, SW12 R1C5, SW13 R2C0, SW14 R2C1, SW15 R2C2, SW16 R2C3, SW17 R2C4, SW18 R2C5, SW19 R0C6, SW2 R0C1, SW20 R1C6, SW21 R2C6, SW22 R3C0, SW23 R3C1, SW24 R3C2, SW25 R3C3, SW26 R3C4, SW27 R3C5, SW28 R4C0, SW29 R4C1, SW3 R0C2, SW30 R4C2, SW31 R4C3, SW32 R4C4, SW33 R4C5, SW34 R5C0, SW35 R5C1, SW36 R5C2, SW37 R5C3, SW38 R5C4, SW39 R5C5, SW4 R0C3, SW40 R3C6, SW41 R4C6, SW42 R5C6, SW43 Power, SW44 Reset, SW5 R0C4, SW6 R0C5, SW7 R1C0, SW8 R1C1, SW9 R1C2, U1 nice!nano v2, U2 SN74LV1T125

Commit message: 0603 resistors and capacitors; rerouted; router rescues stuck signals
- R1-R5, C1, C2 move to KiCad's 0603 hand-solder footprints (README and the
  layout page updated). The last 0805 version is tagged working_0805.
- finish_route.py: when every attempt leaves a signal unrouted, lift one
  neighbouring net in the way, route the connection, reroute the lifted net,
  and keep it only if nothing new is left unrouted. Tracks are removed by
  editing the board file, since removing them through the bindings breaks
  them.
- Both boards: DRC 0 unconnected, schematic parity 0, every pin, the matrix,
  the LED chain and one GND group verified. Gerbers, STEP, renders and plates
  regenerated.

Co-Authored-By: Claude Opus 5.5 <noreply@anthropic.com>
Claude-Session: https://claude.ai/code/session_01D39ubfTYtq6FMvNmmbStTo
Parts:
- C1, C2: footprint Capacitor_SMD:C_0805_2012Metric_Pad1.18x1.45mm_HandSolder -> Capacitor_SMD:C_0603_1608Metric_Pad1.08x0.95mm_HandSolder
- R1, R2, R3, R4, R5: footprint Resistor_SMD:R_0805_2012Metric_Pad1.20x1.40mm_HandSolder -> Resistor_SMD:R_0603_1608Metric_Pad0.98x0.95mm_HandSolder
Routing:
- net GND: track 2697.1 -> 1843.7 mm, vias 237 -> 244
- net COL0: track 374.3 -> 457.8 mm, vias 7 -> 16
- net LED_VDD: track 1040.8 -> 1111.3 mm
- net COL2: track 420.6 -> 362.4 mm
- net /SDA_MOSI: track 77.5 -> 133.5 mm, vias 3 -> 5
- net /LED_EXT: track 131.6 -> 82.9 mm, vias 9 -> 7
- net /P0.24_MISO: track 160.2 -> 116.9 mm
- net /LED_DATA: track 82.9 -> 42.1 mm, vias 8 -> 4
- net /LEDs/LED_D51: track 316.3 -> 357.0 mm, vias 14 -> 4
- net COL4: track 237.0 -> 272.5 mm, vias 14 -> 11
- net ROW5: track 204.6 -> 239.5 mm, vias 5 -> 7
- net ROW2: track 218.2 -> 186.6 mm, vias 9 -> 6
- net COL1: track 387.5 -> 417.5 mm, vias 17 -> 13
- net ROW0: track 249.2 -> 219.5 mm, vias 7 -> 6
- net /SCL_SCK: track 64.0 -> 92.8 mm, vias 3 -> 5
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