File: unicorne.kicad_sch (KiCad schematic)
At the start: 0 parts

Commit message: Add 16° layout, trackpad mock and generated schematic
Layout script derives key positions from crkbd v3-final and places a
TPS43 trackpad and bottom-mounted nice!nano in the centre. The schematic
generator builds the main, key matrix and LED sheets from that layout.

Co-Authored-By: Claude Opus 5.5 <noreply@anthropic.com>
Parts:
- added C1: 10uF, Capacitor_SMD:C_0805_2012Metric, symbol Device:C_Small
- added J1: Battery, Connector_Wire:SolderWire-0.5sqmm_1x02_P4.8mm_D0.9mm_OD2.3mm, symbol Connector_Generic:Conn_01x02
- added J2: TPS43, Connector_PinHeader_2.54mm:PinHeader_1x06_P2.54mm_Vertical, symbol Connector_Generic:Conn_01x06
- added J3: Expansion, Connector_PinHeader_2.54mm:PinHeader_1x06_P2.54mm_Vertical, symbol Connector_Generic:Conn_01x06
- added J4: GPIO, Connector_PinHeader_2.54mm:PinHeader_1x04_P2.54mm_Vertical, symbol Connector_Generic:Conn_01x04
- added JP1: LED data, Jumper:SolderJumper-2_P1.3mm_Open_RoundedPad1.0x1.5mm, symbol Jumper:SolderJumper_2_Open
- added Q1: AO3401A, Package_TO_SOT_SMD:SOT-23, symbol Transistor_FET:AO3401A
- added Q2: 2N7002, Package_TO_SOT_SMD:SOT-23, symbol Transistor_FET:2N7002
- added R1, R2: 100k, Resistor_SMD:R_0603_1608Metric, symbol Device:R_Small
- added R3, R4: 4.7k, Resistor_SMD:R_0603_1608Metric, symbol Device:R_Small
- added R5: 10k, Resistor_SMD:R_0603_1608Metric, symbol Device:R_Small
- added SW43: Power, Button_Switch_SMD:SW_SPDT_Shouhan_MSK12C02, symbol Switch:SW_SPDT
- added SW44: Reset, Button_Switch_SMD:SW_SPST_TL3342, symbol Switch:SW_Push
- added U1: nice!nano v2, unicorne:nice_nano, symbol unicorne:nice_nano_v2
Connections:
- new net +3V3: J2.3 (Pin_3), J3.1 (Pin_1), R3.1, R4.1, R5.1, U1.21 (VCC)
- new net BATT+: J1.1 (Pin_1), SW43.2 (B)
- new net COL0: U1.17 (P1.15/D18)
- new net COL1: U1.16 (P1.13/D15)
- new net COL2: U1.15 (P1.11/D14)
- new net COL3: U1.14 (P0.10/D16)
- new net COL4: U1.13 (P0.09/D10)
- new net COL5: U1.31 (P1.01)
- new net COL6: U1.32 (P1.02)
- new net GND: C1.2, J1.2 (Pin_2), J2.4 (Pin_4), J3.2 (Pin_2), J4.1 (Pin_1), Q2.2 (S), R2.2, SW44.2, U1.23 (GND), U1.3 (GND), U1.4 (GND)
- new net LED_DIN: JP1.2 (B)
- new net LED_EN: J4.3 (Pin_3), Q2.1 (G), R2.1, U1.9 (P1.00/D6)
- new net LED_EN_N: Q1.1 (G), Q2.3 (D), R1.2
- new net LED_VDD: C1.1, Q1.3 (D)
- new net P0.06: J3.4 (Pin_4), JP1.1 (A), U1.1 (P0.06/D1)
- new net P0.08: J3.3 (Pin_3), U1.2 (P0.08/D0)
- new net P0.11: J4.4 (Pin_4), U1.10 (P0.11/D7)
- new net P0.24: J4.2 (Pin_2), U1.8 (P0.24/D5)
- new net ROW0: U1.20 (P0.31/D21)
- new net ROW1: U1.19 (P0.29/D20)
- new net ROW2: U1.18 (P0.02/D19)
- new net ROW3: U1.11 (P1.04/D8)
- new net ROW4: U1.12 (P1.06/D9)
- new net ROW5: U1.33 (P1.07)
- new net RST: SW44.1, U1.22 (RST)
- new net SCL: J2.2 (Pin_2), J3.6 (Pin_6), R4.2, U1.6 (P0.20/D3)
- new net SDA: J2.1 (Pin_1), J3.5 (Pin_5), R3.2, U1.5 (P0.17/D2)
- new net TP_NRST: J2.5 (Pin_5), R5.2
- new net TP_RDY: J2.6 (Pin_6), U1.7 (P0.22/D4)
- new net VBAT: Q1.2 (S), R1.1, SW43.1 (A), U1.24 (RAW/B+)
- no-connect marks 0 -> 1
Other:
- added sheet Key matrix (matrix.kicad_sch)
- added sheet LEDs (leds.kicad_sch)
- note added: "Battery: J1 pads -> power switch -> nice!nano RAW/B+. With the switch off the battery is disconnected; USB still powers the board."
- note added: "J3 expansion: UART on P0.08/P0.06, I2C shared with the trackpad. J4 GPIO: P0.24 and P0.11 free; P1.00 is LED_EN."
- note added: "LED supply: Q1 switches battery voltage onto LED_VDD when P1.00 (LED_EN) is high. R1/R2 keep it off during boot. ZMK: ext-power on P1.00 for the LEDs only; VCC (trackpad, header) stays on. Close JP1 to drive the LEDs from P0.06."
- note added: "Trackpad: Azoteq TPS43 (IQS572), I2C at 1.65-3.6 V. J2 is six bare pads for short wires to the module's own pads (no FPC, keeps it thin), in the module's order: SDA, SCL, 3V3, GND, RST, RDY (datasheet v1.06, figure 2.1)."
- note added: "nice!nano v2, mounted on the bottom side under the trackpad. Pins 31-33 are the three inner pads (low-frequency GPIO), used for the matrix. P0.09 / P0.10 are NFC pins: ZMK needs CONFIG_NFCT_PINS_AS_GPIOS=y."
- company: (none) -> unicorne

Commit message: Use a 6x6x5 mm through-hole tactile switch for reset
Co-Authored-By: Claude Opus 5.5 <noreply@anthropic.com>
Parts:
- SW44: footprint Button_Switch_SMD:SW_SPST_TL3342 -> Button_Switch_THT:SW_PUSH_6mm_H5mm
Changed lines of the file:
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@@
 		(instances
 			(project "unicorne"
-				(path "/7e94b886-8de9-4278-978e-e3916245dcb2"
+				(path "/452a8a2e-cfaa-4649-b7eb-908632b76421"
 					(reference "U1")
 					(unit 1)
@@
 		(instances
 			(project "unicorne"
-				(path "/7e94b886-8de9-4278-978e-e3916245dcb2"
+				(path "/452a8a2e-cfaa-4649-b7eb-908632b76421"
 					(reference "#PWRU01")
 					(unit 1)
@@
 		(instances
 			(project "unicorne"
-				(path "/7e94b886-8de9-4278-978e-e3916245dcb2"
+				(path "/452a8a2e-cfaa-4649-b7eb-908632b76421"
 					(reference "#PWRU02")
 					(unit 1)
@@
 		(instances
 			(project "unicorne"
-				(path "/7e94b886-8de9-4278-978e-e3916245dcb2"
+				(path "/452a8a2e-cfaa-4649-b7eb-908632b76421"
 					(reference "#PWRU03")
 					(unit 1)
@@
 		(instances
 			(project "unicorne"
-				(path "/7e94b886-8de9-4278-978e-e3916245dcb2"
+				(path "/452a8a2e-cfaa-4649-b7eb-908632b76421"
 					(reference "#PWRU04")
 					(unit 1)
@@
 		(instances
 			(project "unicorne"
-				(path "/7e94b886-8de9-4278-978e-e3916245dcb2"
+				(path "/452a8a2e-cfaa-4649-b7eb-908632b76421"
 					(reference "J1")
 					(unit 1)
@@
 		(instances
 			(project "unicorne"
-				(path "/7e94b886-8de9-4278-978e-e3916245dcb2"
+				(path "/452a8a2e-cfaa-4649-b7eb-908632b76421"
 					(reference "#PWRU05")
 					(unit 1)
@@
 		(instances
 			(project "unicorne"
-				(path "/7e94b886-8de9-4278-978e-e3916245dcb2"
+				(path "/452a8a2e-cfaa-4649-b7eb-908632b76421"
 					(reference "SW43")
 					(unit 1)
@@
 			)
 		)
-		(property "Footprint" "Button_Switch_SMD:SW_SPST_TL3342"
+		(property "Footprint" "Button_Switch_THT:SW_PUSH_6mm_H5mm"
 			(at 76.2 66.04 0)
 			(effects
@@
 		(instances
 			(project "unicorne"
-				(path "/7e94b886-8de9-4278-978e-e3916245dcb2"
+				(path "/452a8a2e-cfaa-4649-b7eb-908632b76421"
 					(reference "SW44")
 					(unit 1)
@@
 		(instances
 			(project "unicorne"
-				(path "/7e94b886-8de9-4278-978e-e3916245dcb2"
+				(path "/452a8a2e-cfaa-4649-b7eb-908632b76421"
 					(reference "#PWRU06")
 					(unit 1)
@@
 		(instances
 			(project "unicorne"
-				(path "/7e94b886-8de9-4278-978e-e3916245dcb2"
+				(path "/452a8a2e-cfaa-4649-b7eb-908632b76421"
 					(reference "Q1")
 					(unit 1)
@@
 		(instances
 			(project "unicorne"
-				(path "/7e94b886-8de9-4278-978e-e3916245dcb2"
+				(path "/452a8a2e-cfaa-4649-b7eb-908632b76421"
 					(reference "#PWRU07")
 					(unit 1)
@@
 		(instances
 			(project "unicorne"
-				(path "/7e94b886-8de9-4278-978e-e3916245dcb2"
+				(path "/452a8a2e-cfaa-4649-b7eb-908632b76421"
 					(reference "Q2")
 					(unit 1)
@@
 		(instances
 			(project "unicorne"
-				(path "/7e94b886-8de9-4278-978e-e3916245dcb2"
+				(path "/452a8a2e-cfaa-4649-b7eb-908632b76421"
 					(reference "#PWRU08")
 					(unit 1)
@@
 		(instances
 			(project "unicorne"
-				(path "/7e94b886-8de9-4278-978e-e3916245dcb2"
+				(path "/452a8a2e-cfaa-4649-b7eb-908632b76421"
 					(reference "R1")
 					(unit 1)
@@
 		(instances
 			(project "unicorne"
-				(path "/7e94b886-8de9-4278-978e-e3916245dcb2"
+				(path "/452a8a2e-cfaa-4649-b7eb-908632b76421"
 					(reference "R2")
 					(unit 1)
@@
 		(instances
 			(project "unicorne"
-				(path "/7e94b886-8de9-4278-978e-e3916245dcb2"
+				(path "/452a8a2e-cfaa-4649-b7eb-908632b76421"
 					(reference "#PWRU09")
 					(unit 1)
@@
 		(instances
 			(project "unicorne"
-				(path "/7e94b886-8de9-4278-978e-e3916245dcb2"
+				(path "/452a8a2e-cfaa-4649-b7eb-908632b76421"
 					(reference "C1")
 					(unit 1)
@@
 		(instances
 			(project "unicorne"
-				(path "/7e94b886-8de9-4278-978e-e3916245dcb2"
+				(path "/452a8a2e-cfaa-4649-b7eb-908632b76421"
 					(reference "#PWRU10")
 					(unit 1)
@@
 		(instances
 			(project "unicorne"
-				(path "/7e94b886-8de9-4278-978e-e3916245dcb2"
+				(path "/452a8a2e-cfaa-4649-b7eb-908632b76421"
 					(reference "#PWRU11")
 					(unit 1)
@@
 		(instances
 			(project "unicorne"
-				(path "/7e94b886-8de9-4278-978e-e3916245dcb2"
+				(path "/452a8a2e-cfaa-4649-b7eb-908632b76421"
 					(reference "JP1")
 					(unit 1)
@@
 		(instances
 			(project "unicorne"
-				(path "/7e94b886-8de9-4278-978e-e3916245dcb2"
+				(path "/452a8a2e-cfaa-4649-b7eb-908632b76421"
 					(reference "J2")
 					(unit 1)
@@
 		(instances
 			(project "unicorne"
-				(path "/7e94b886-8de9-4278-978e-e3916245dcb2"
+				(path "/452a8a2e-cfaa-4649-b7eb-908632b76421"
 					(reference "#PWRU12")
 					(unit 1)
@@
 		(instances
 			(project "unicorne"
-				(path "/7e94b886-8de9-4278-978e-e3916245dcb2"
+				(path "/452a8a2e-cfaa-4649-b7eb-908632b76421"
 					(reference "#PWRU13")
 					(unit 1)
@@
 		(instances
 			(project "unicorne"
-				(path "/7e94b886-8de9-4278-978e-e3916245dcb2"
+				(path "/452a8a2e-cfaa-4649-b7eb-908632b76421"
 					(reference "R3")
 					(unit 1)
@@
 		(instances
 			(project "unicorne"
-				(path "/7e94b886-8de9-4278-978e-e3916245dcb2"
+				(path "/452a8a2e-cfaa-4649-b7eb-908632b76421"
 					(reference "#PWRU14")
 					(unit 1)
@@
 		(instances
 			(project "unicorne"
-				(path "/7e94b886-8de9-4278-978e-e3916245dcb2"
+				(path "/452a8a2e-cfaa-4649-b7eb-908632b76421"
 					(reference "R4")
 					(unit 1)
@@
 		(instances
 			(project "unicorne"
-				(path "/7e94b886-8de9-4278-978e-e3916245dcb2"
+				(path "/452a8a2e-cfaa-4649-b7eb-908632b76421"
 					(reference "#PWRU15")
 					(unit 1)
@@
 		(instances
 			(project "unicorne"
-				(path "/7e94b886-8de9-4278-978e-e3916245dcb2"
+				(path "/452a8a2e-cfaa-4649-b7eb-908632b76421"
 					(reference "R5")
 					(unit 1)
@@
 		(instances
 			(project "unicorne"
-				(path "/7e94b886-8de9-4278-978e-e3916245dcb2"
+				(path "/452a8a2e-cfaa-4649-b7eb-908632b76421"
 					(reference "#PWRU16")
 					(unit 1)
@@
 		(instances
 			(project "unicorne"
-				(path "/7e94b886-8de9-4278-978e-e3916245dcb2"
+				(path "/452a8a2e-cfaa-4649-b7eb-908632b76421"
 					(reference "J3")
 					(unit 1)
@@
 		(instances
 			(project "unicorne"
-				(path "/7e94b886-8de9-4278-978e-e3916245dcb2"
+				(path "/452a8a2e-cfaa-4649-b7eb-908632b76421"
 					(reference "#PWRU17")
 					(unit 1)
@@
 		(instances
 			(project "unicorne"
-				(path "/7e94b886-8de9-4278-978e-e3916245dcb2"
+				(path "/452a8a2e-cfaa-4649-b7eb-908632b76421"
 					(reference "#PWRU18")
 					(unit 1)
@@
 		(instances
 			(project "unicorne"
-				(path "/7e94b886-8de9-4278-978e-e3916245dcb2"
+				(path "/452a8a2e-cfaa-4649-b7eb-908632b76421"
 					(reference "J4")
 					(unit 1)
@@
 		(instances
 			(project "unicorne"
-				(path "/7e94b886-8de9-4278-978e-e3916245dcb2"
+				(path "/452a8a2e-cfaa-4649-b7eb-908632b76421"
 					(reference "#PWRU19")
 					(unit 1)
@@
 		(instances
 			(project "unicorne"
-				(path "/7e94b886-8de9-4278-978e-e3916245dcb2"
+				(path "/452a8a2e-cfaa-4649-b7eb-908632b76421"
 					(reference "#FLGU20")
 					(unit 1)
@@
 		(instances
 			(project "unicorne"
-				(path "/7e94b886-8de9-4278-978e-e3916245dcb2"
+				(path "/452a8a2e-cfaa-4649-b7eb-908632b76421"
 					(reference "#PWRU21")
 					(unit 1)
@@
 		(instances
 			(project "unicorne"
-				(path "/7e94b886-8de9-4278-978e-e3916245dcb2"
+				(path "/452a8a2e-cfaa-4649-b7eb-908632b76421"
 					(reference "#FLGU22")
 					(unit 1)
@@
 		(instances
 			(project "unicorne"
-				(path "/7e94b886-8de9-4278-978e-e3916245dcb2"
+				(path "/452a8a2e-cfaa-4649-b7eb-908632b76421"
 					(reference "#FLGU23")
 					(unit 1)
@@
 		(instances
 			(project "unicorne"
-				(path "/7e94b886-8de9-4278-978e-e3916245dcb2"
+				(path "/452a8a2e-cfaa-4649-b7eb-908632b76421"
 					(reference "#PWRU24")
 					(unit 1)
@@
 		(instances
 			(project "unicorne"
-				(path "/7e94b886-8de9-4278-978e-e3916245dcb2"
+				(path "/452a8a2e-cfaa-4649-b7eb-908632b76421"
 					(reference "#FLGU25")
 					(unit 1)
@@
 		(instances
 			(project "unicorne"
-				(path "/7e94b886-8de9-4278-978e-e3916245dcb2"
+				(path "/452a8a2e-cfaa-4649-b7eb-908632b76421"
 					(page "2")
 				)
@@
 		(instances
 			(project "unicorne"
-				(path "/7e94b886-8de9-4278-978e-e3916245dcb2"
+				(path "/452a8a2e-cfaa-4649-b7eb-908632b76421"
 					(page "3")
 				)

Commit message: Place MX and Choc PCBs from the layout and schematic
gen_pcb.py builds both boards: switches, diodes and LEDs from Corne v3
offsets, the nice!nano flush on the bottom, centre parts, outline,
36-key break lines with mouse bites, M2 holes, pad labels and a
nice!nano pin table on the silkscreen. Adds TPS43 / PAW3395-PMW3360
sensor pads and a 6x6 THT reset switch; underglow becomes SK6812MINI.

Co-Authored-By: Claude Opus 5.5 <noreply@anthropic.com>
Parts:
- added J5: PAW3395 / PMW3360, Connector_PinHeader_2.54mm:PinHeader_1x08_P2.54mm_Vertical, symbol Connector_Generic:Conn_01x08
- J1: Note (none) -> Through-hole B+ / B- pads, reachable from both sides; now left out of the parts list
- J2: Note (none) -> Bare pads for wires to the TPS43, in the module's pad order; now left out of the parts list
- JP1: now left out of the parts list
- SW43: Note (none) -> Battery cut-off slide switch (part to confirm)
Connections:
- net +3V3: now also J5.1 (Pin_1)
- net GND: now also J5.2 (Pin_2)
- net P0.11 renamed P0.11_CS
- net P0.11_CS: now also J5.6 (Pin_6)
- net P0.24 renamed P0.24_MISO
- net P0.24_MISO: now also J5.5 (Pin_5)
- net SCL renamed SCL_SCK
- net SCL_SCK: now also J5.3 (Pin_3)
- net SDA renamed SDA_MOSI
- net SDA_MOSI: now also J5.4 (Pin_4)
- net TP_NRST renamed NRST
- net NRST: now also J5.8 (Pin_8)
- net TP_RDY renamed RDY_MOTION
- net RDY_MOTION: now also J5.7 (Pin_7)
Other:
- note added: "J3 expansion: UART on P0.08/P0.06, I2C shared with the trackpad. J4 GPIO: P0.24 and P0.11 (sensor MISO/CS if J5 is used); P1.00 is LED_EN."
- note added: "J5: optical sensor (PAW3395 / PMW3360) instead of the trackpad, over SPI: SCK = P0.20, MOSI = P0.17, MISO = P0.24, CS = P0.11, MOTION = P0.22, RST = NRST. SCK/MOSI/MOTION share the trackpad's SCL/SDA/RDY: fit one or the other, and leave R3/R4 off with a sensor. Check the sensor board's supply: some want 5 V."
- note removed: "J3 expansion: UART on P0.08/P0.06, I2C shared with the trackpad. J4 GPIO: P0.24 and P0.11 free; P1.00 is LED_EN."
