File: leds.kicad_sch (KiCad schematic)
At the start: 54 parts

Commit message: Place MX and Choc PCBs from the layout and schematic
gen_pcb.py builds both boards: switches, diodes and LEDs from Corne v3
offsets, the nice!nano flush on the bottom, centre parts, outline,
36-key break lines with mouse bites, M2 holes, pad labels and a
nice!nano pin table on the silkscreen. Adds TPS43 / PAW3395-PMW3360
sensor pads and a 6x6 THT reset switch; underglow becomes SK6812MINI.

Co-Authored-By: Claude Opus 5.5 <noreply@anthropic.com>
Parts:
- removed LED1, LED10, LED11, LED12, LED2, LED3, LED4, LED5, LED6, LED7, LED8, LED9: WS2812B, LED_SMD:LED_WS2812B_PLCC4_5.0x5.0mm_P3.2mm, symbol LED:WS2812B
- added LED1, LED10, LED11, LED12, LED2, LED3, LED4, LED5, LED6, LED7, LED8, LED9: SK6812MINI, LED_SMD:LED_SK6812MINI_PLCC4_3.5x3.5mm_P1.75mm, symbol LED:SK6812MINI
Connections:
- net GND: now also LED1.2 (VSS), LED10.2 (VSS), LED11.2 (VSS), LED12.2 (VSS), LED2.2 (VSS), LED3.2 (VSS), LED4.2 (VSS), LED5.2 (VSS), LED6.2 (VSS), LED7.2 (VSS), LED8.2 (VSS), LED9.2 (VSS)
- net LED_D1: now also LED1.1 (DOUT), LED2.3 (DIN)
- net LED_D10: now also LED10.1 (DOUT), LED11.3 (DIN)
- net LED_D11: now also LED11.1 (DOUT), LED12.3 (DIN)
- net LED_D12: now also LED12.1 (DOUT)
- net LED_D2: now also LED2.1 (DOUT), LED3.3 (DIN)
- net LED_D3: now also LED3.1 (DOUT), LED4.3 (DIN)
- net LED_D4: now also LED4.1 (DOUT), LED5.3 (DIN)
- net LED_D5: now also LED5.1 (DOUT), LED6.3 (DIN)
- net LED_D6: now also LED6.1 (DOUT), LED7.3 (DIN)
- net LED_D7: now also LED7.1 (DOUT), LED8.3 (DIN)
- net LED_D8: now also LED8.1 (DOUT), LED9.3 (DIN)
- net LED_D9: now also LED10.3 (DIN), LED9.1 (DOUT)
- net LED_DIN: now also LED1.3 (DIN)
- net LED_VDD: now also LED1.4 (VDD), LED10.4 (VDD), LED11.4 (VDD), LED12.4 (VDD), LED2.4 (VDD), LED3.4 (VDD), LED4.4 (VDD), LED5.4 (VDD), LED6.4 (VDD), LED7.4 (VDD), LED8.4 (VDD), LED9.4 (VDD)
Other:
- note added: "Chain: LED1-12 underglow (SK6812MINI, bottom), LED13-48 per-key on the inner five columns and thumbs, LED49-54 the breakable outer pinky columns last. Every LED runs from LED_VDD."
- note removed: "Chain: LED1-12 underglow (WS2812B, bottom), LED13-48 per-key on the inner five columns and thumbs, LED49-54 the breakable outer pinky columns last. Every LED runs from LED_VDD."

Commit message: Rework LED power, break lines and centre placement; add routing tools
- LED supply chosen by solder jumper JP2: nice!nano VCC, or an external
  supply on new LED IN pads (J6); never the battery pin. SN74LV1T125
  level shifter (U2) with bypass jumper JP3.
- Centre parts rearranged so the nice!nano's matrix pins are clear.
- 0805 hand-solder passives; LED chain runs left to right per row.
- Break lines: no sliver slots, perforated end to end, tabs over the lanes.
- Mounting holes stay inside the board and off the routing lanes.
- Routing tools (lanes, Freerouting driver, maze router) and placeholder
  STEP models. Boards are committed placed but unrouted.

Co-Authored-By: Claude Opus 5.5 <noreply@anthropic.com>
Parts:
- LED18: Key L K15 -> L K11
- LED19: Key L K14 -> L K12
- LED21: Key L K12 -> L K14
- LED22: Key L K11 -> L K15
- LED31: Key R K01 -> R K05
- LED32: Key R K02 -> R K04
- LED34: Key R K04 -> R K02
- LED35: Key R K05 -> R K01
- LED41: Key R K21 -> R K25
- LED42: Key R K22 -> R K24
- LED44: Key R K24 -> R K22
- LED45: Key R K25 -> R K21

Commit message: Route the MX board
finish_route.py lays fixed lanes on the key grid (columns on top; rows,
LED data and LED supply on the bottom), then routes KiCad's remaining
ratsnest with the maze router, pours GND on both layers and stitches
them. DRC: 0 unconnected, 0 copper violations, matches the schematic.

LED chain reordered to cross the board once; Q1 rotated so its source
faces JP2.

Co-Authored-By: Claude Opus 5.5 <noreply@anthropic.com>
Parts:
- removed LED10, LED11, LED12, LED7, LED8, LED9: SK6812MINI, LED_SMD:LED_SK6812MINI_PLCC4_3.5x3.5mm_P1.75mm, symbol LED:SK6812MINI
- removed LED43, LED44, LED45, LED46, LED47, LED48: SK6812MINI-E, LED_SMD:LED_SK6812MINI-E_3.2x2.8mm_P1.5mm_ReverseMount, symbol LED:SK6812MINI-E
- added LED10, LED11, LED12, LED7, LED8, LED9: SK6812MINI-E, LED_SMD:LED_SK6812MINI-E_3.2x2.8mm_P1.5mm_ReverseMount, symbol LED:SK6812MINI-E
- added LED43, LED44, LED45, LED46, LED47, LED48: SK6812MINI, LED_SMD:LED_SK6812MINI_PLCC4_3.5x3.5mm_P1.75mm, symbol LED:SK6812MINI
- LED1: Key L UG0 -> L UG5
- LED13: Key L K01 -> L K12
- LED14: Key L K02 -> L K13
- LED15: Key L K03 -> L K14
- LED16: Key L K04 -> L K15
- LED17: Key L K05 -> L K21
- LED18: Key L K11 -> L K22
- LED19: Key L K12 -> L K23
- LED2: Key L UG1 -> L UG2
- LED20: Key L K13 -> L K24
- LED21: Key L K14 -> L K25
- LED22: Key L K15 -> L T0
- LED23: Key L K21 -> L T1
- LED24: Key L K22 -> L T2
- LED25: Key L K23 -> R T2
- LED26: Key L K24 -> R T1
- LED27: Key L K25 -> R T0
- LED28: Key L T0 -> R K05
- LED29: Key L T1 -> R K04
- LED3: Key L UG2 -> L UG4
- LED30: Key L T2 -> R K03
- LED31: Key R K05 -> R K02
- LED32: Key R K04 -> R K01
- LED33: Key R K03 -> R K15
- LED34: Key R K02 -> R K14
- LED35: Key R K01 -> R K13
- LED36: Key R K15 -> R K12
- LED37: Key R K14 -> R K11
- LED38: Key R K13 -> R K25
- LED39: Key R K12 -> R K24
- LED4: Key L UG3 -> L UG1
- LED40: Key R K11 -> R K23
- LED41: Key R K25 -> R K22
- LED42: Key R K24 -> R K21
- LED49: Key L K00 -> R K00
- LED5: Key L UG4 -> L UG3
- LED50: Key L K10 -> R K10
- LED51: Key L K20 -> R K20
- LED52: Key R K00 -> L K00
- LED53: Key R K10 -> L K10
- LED54: Key R K20 -> L K20
- LED6: Key L UG5 -> L UG0
Connections:
- net GND: now also LED10.1 (VSS), LED11.1 (VSS), LED12.1 (VSS), LED43.2 (VSS), LED44.2 (VSS), LED45.2 (VSS), LED46.2 (VSS), LED47.2 (VSS), LED48.2 (VSS), LED7.1 (VSS), LED8.1 (VSS), LED9.1 (VSS)
- net LED_D10: now also LED10.4 (DOUT), LED11.2 (DIN)
- net LED_D11: now also LED11.4 (DOUT), LED12.2 (DIN)
- net LED_D12: now also LED12.4 (DOUT)
- net LED_D42: now also LED43.3 (DIN)
- net LED_D43: now also LED43.1 (DOUT), LED44.3 (DIN)
- net LED_D44: now also LED44.1 (DOUT), LED45.3 (DIN)
- net LED_D45: now also LED45.1 (DOUT), LED46.3 (DIN)
- net LED_D46: now also LED46.1 (DOUT), LED47.3 (DIN)
- net LED_D47: now also LED47.1 (DOUT), LED48.3 (DIN)
- net LED_D48: now also LED48.1 (DOUT)
- net LED_D6: now also LED7.2 (DIN)
- net LED_D7: now also LED7.4 (DOUT), LED8.2 (DIN)
- net LED_D8: now also LED8.4 (DOUT), LED9.2 (DIN)
- net LED_D9: now also LED10.2 (DIN), LED9.4 (DOUT)
- net LED_VDD: now also LED10.3 (VDD), LED11.3 (VDD), LED12.3 (VDD), LED43.4 (VDD), LED44.4 (VDD), LED45.4 (VDD), LED46.4 (VDD), LED47.4 (VDD), LED48.4 (VDD), LED7.3 (VDD), LED8.3 (VDD), LED9.3 (VDD)
Other:
- note added: "Chain: left underglow, left rows (left to right), left thumbs, right thumbs, right rows, right underglow, then the breakable outer pinky columns (right, then left). LED_VDD powers all."
- note removed: "Chain: LED1-12 underglow (SK6812MINI, bottom), LED13-48 per-key on the inner five columns and thumbs, LED49-54 the breakable outer pinky columns last. Every LED runs from LED_VDD."

Commit message: Add 3D models and STEP export
Project footprints point at models in lib/3d/: Kailh MX and Choc hotswap
sockets and the Choc V1 switch (keyswitch-kicad-library), plus placeholder
boxes for the nice!nano, TPS43, MX switch, SK6812MINI and MSK-12C02 (the
last two copied from the stock library with a model added). The trackpad
model sits on a board-only footprint; bare pads carry no model.
export_3d.py writes export/unicorne-{mx,choc}.step; renders alongside.

Both boards regenerated and re-routed: DRC 0 unconnected, 0 copper
violations.

Co-Authored-By: Claude Opus 5.5 <noreply@anthropic.com>
Parts:
- LED1, LED2, LED3, LED4, LED43, LED44, LED45, LED46, LED47, LED48, LED5, LED6: footprint LED_SMD:LED_SK6812MINI_PLCC4_3.5x3.5mm_P1.75mm -> unicorne:LED_SK6812MINI_PLCC4_3.5x3.5mm_P1.75mm
