File: leds.kicad_sch (KiCad schematic)
At the start: 54 parts

Commit message: Route both boards with KiCadRoutingTools; no vias in pads
tools/krt_route.py: fixed lanes, then KiCadRoutingTools 0.23.7 for every other
signal at standard JLCPCB sizes (0.6/0.3 vias, 0.2 tracks) with no via in or next
to a pad, own net's included; the maze router for any net it could only finish
with undersized vias; GND pours and stitching; its plane repair; then any via
touching a pad is removed. The tools relax the project's rules on disk: ours are
put back.

MX lanes: LED_VDD's jog across a break line moves from 5.5 to 4.5 mm off the
line. At 5.5 it boxed in the outer-column LED DIN pads, so 8 LED data links had
no room for a via outside a pad. Lane-only board: no DRC errors.

Stitching vias (finish_route.stitch) and our maze router stay off SMD pads too.
The previous MX board had 82 vias in pads, now none on either board.

MX: U2 pad 3 (GND) is boxed in by LED_DIN; joined by hand with a via between
pads 3 and 4 (noted in the README).

Both boards: DRC 0 unconnected, 0 copper violations, schematic parity clean;
all 482 schematic pins, 42 keys and the 54-LED chain check out pin by pin.
Waves, LED map, plates, gerbers, STEP and renders regenerated.

Co-Authored-By: Claude Opus 5.5 <noreply@anthropic.com>
Claude-Session: https://claude.ai/code/session_01D39ubfTYtq6FMvNmmbStTo
Parts:
- removed LED1, LED2, LED3, LED43, LED44, LED46, LED48, LED5, LED6: SK6812MINI, unicorne:LED_SK6812MINI_PLCC4_3.5x3.5mm_P1.75mm, symbol LED:SK6812MINI
- removed LED11, LED13, LED18, LED23, LED26, LED29, LED37, LED40, LED8: SK6812MINI-E, LED_SMD:LED_SK6812MINI-E_3.2x2.8mm_P1.5mm_ReverseMount, symbol LED:SK6812MINI-E
- added LED1, LED2, LED3, LED43, LED44, LED46, LED48, LED5, LED6: SK6812MINI-E, LED_SMD:LED_SK6812MINI-E_3.2x2.8mm_P1.5mm_ReverseMount, symbol LED:SK6812MINI-E
- added LED11, LED13, LED18, LED23, LED26, LED29, LED37, LED40, LED8: SK6812MINI, unicorne:LED_SK6812MINI_PLCC4_3.5x3.5mm_P1.75mm, symbol LED:SK6812MINI
- LED10: Key L K04 -> L K21
- LED14: Key L K13 -> L K01
- LED15: Key L K14 -> L K02
- LED16: Key L K15 -> L K12
- LED17: Key L K21 -> L K13
- LED19: Key L K23 -> L K03
- LED20: Key L K24 -> L K04
- LED21: Key L K25 -> L K14
- LED22: Key L T0 -> L K15
- LED24: Key L T2 -> L K05
- LED25: Key R T2 -> R K05
- LED27: Key R T0 -> R K15
- LED28: Key R K05 -> R K25
- LED30: Key R K03 -> R T2
- LED31: Key R K02 -> R T1
- LED32: Key R K01 -> R T0
- LED33: Key R K15 -> R K24
- LED35: Key R K13 -> R K04
- LED36: Key R K12 -> R K03
- LED38: Key R K25 -> R K13
- LED39: Key R K24 -> R K23
- LED4: Key L UG1 -> L UG5
- LED42: Key R K21 -> R K12
- LED45: Key R UG5 -> R UG0
- LED47: Key R UG1 -> R UG3
- LED49: Key R K00 -> R K20
- LED51: Key R K20 -> R K00
- LED7: Key L K01 -> L K23
- LED9: Key L K03 -> L K22
Connections:
- net GND: now also LED1.1 (VSS), LED11.2 (VSS), LED13.2 (VSS), LED18.2 (VSS), LED2.1 (VSS), LED23.2 (VSS), LED26.2 (VSS), LED29.2 (VSS), LED3.1 (VSS), LED37.2 (VSS), LED40.2 (VSS), LED43.1 (VSS), LED44.1 (VSS), LED46.1 (VSS), LED48.1 (VSS), LED5.1 (VSS), LED6.1 (VSS), LED8.2 (VSS)
- net LED_D1: now also LED1.4 (DOUT), LED2.2 (DIN)
- net LED_D10: now also LED11.3 (DIN)
- net LED_D11: now also LED11.1 (DOUT)
- net LED_D12: now also LED13.3 (DIN)
- net LED_D13: now also LED13.1 (DOUT)
- net LED_D17: now also LED18.3 (DIN)
- net LED_D18: now also LED18.1 (DOUT)
- net LED_D2: now also LED2.4 (DOUT), LED3.2 (DIN)
- net LED_D22: now also LED23.3 (DIN)
- net LED_D23: now also LED23.1 (DOUT)
- net LED_D25: now also LED26.3 (DIN)
- net LED_D26: now also LED26.1 (DOUT)
- net LED_D28: now also LED29.3 (DIN)
- net LED_D29: now also LED29.1 (DOUT)
- net LED_D3: now also LED3.4 (DOUT)
- net LED_D36: now also LED37.3 (DIN)
- net LED_D37: now also LED37.1 (DOUT)
- net LED_D39: now also LED40.3 (DIN)
- net LED_D4: now also LED5.2 (DIN)
- net LED_D40: now also LED40.1 (DOUT)
- net LED_D42: now also LED43.2 (DIN)
- net LED_D43: now also LED43.4 (DOUT), LED44.2 (DIN)
- net LED_D44: now also LED44.4 (DOUT)
- net LED_D45: now also LED46.2 (DIN)
- net LED_D46: now also LED46.4 (DOUT)
- net LED_D47: now also LED48.2 (DIN)
- net LED_D48: now also LED48.4 (DOUT)
- net LED_D5: now also LED5.4 (DOUT), LED6.2 (DIN)
- net LED_D6: now also LED6.4 (DOUT)
- net LED_D7: now also LED8.3 (DIN)
- net LED_D8: now also LED8.1 (DOUT)
- net LED_DIN: now also LED1.2 (DIN)
- net LED_VDD: now also LED1.3 (VDD), LED11.4 (VDD), LED13.4 (VDD), LED18.4 (VDD), LED2.3 (VDD), LED23.4 (VDD), LED26.4 (VDD), LED29.4 (VDD), LED3.3 (VDD), LED37.4 (VDD), LED40.4 (VDD), LED43.3 (VDD), LED44.3 (VDD), LED46.3 (VDD), LED48.3 (VDD), LED5.3 (VDD), LED6.3 (VDD), LED8.4 (VDD)
