File: export/quilter/mx/fallback/unicorne.kicad_pcb (KiCad board)
At the start: 2 copper layers, 293.4 x 118.8 mm, 175 parts, among them J1 Battery, J2 TPS43, J3 Expansion, J4 GPIO, J5 PAW3395 / PMW3360, J6 LED power in, Q1 AO3401A, Q2 2N7002, SW1 R0C0, SW10 R1C3, SW11 R1C4, SW12 R1C5, SW13 R2C0, SW14 R2C1, SW15 R2C2, SW16 R2C3, SW17 R2C4, SW18 R2C5, SW19 R0C6, SW2 R0C1, SW20 R1C6, SW21 R2C6, SW22 R3C0, SW23 R3C1, SW24 R3C2, SW25 R3C3, SW26 R3C4, SW27 R3C5, SW28 R4C0, SW29 R4C1, SW3 R0C2, SW30 R4C2, SW31 R4C3, SW32 R4C4, SW33 R4C5, SW34 R5C0, SW35 R5C1, SW36 R5C2, SW37 R5C3, SW38 R5C4, SW39 R5C5, SW4 R0C3, SW40 R3C6, SW41 R4C6, SW42 R5C6, SW43 Power, SW44 Reset, SW5 R0C4, SW6 R0C5, SW7 R1C0, SW8 R1C1, SW9 R1C2, U1 nice!nano v2, U2 SN74LV1T125

Commit message: Add Linux KiCad path support, host tests and setup notes
Co-Authored-By: Claude Opus 5 <noreply@anthropic.com>
Routing:
- net LED_VDD: track 704.5 -> 0.00 mm
- net ROW3: track 106.6 -> 0.00 mm
- net ROW4: track 106.6 -> 0.00 mm
- net ROW1: track 106.6 -> 0.00 mm
- net ROW0: track 106.6 -> 0.00 mm
- net ROW5: track 106.6 -> 0.00 mm
- net ROW2: track 106.6 -> 0.00 mm
- net COL4: track 87.6 -> 0.00 mm, vias 6 -> 0
- net COL2: track 87.6 -> 0.00 mm, vias 6 -> 0
- net COL3: track 87.6 -> 0.00 mm, vias 6 -> 0
- net COL1: track 87.6 -> 0.00 mm, vias 6 -> 0
- net COL0: track 87.6 -> 0.00 mm, vias 6 -> 0
- net COL5: track 87.6 -> 0.00 mm, vias 6 -> 0
- net GND: track 30.6 -> 0.00 mm, vias 36 -> 0
- net /LEDs/LED_D14: track 18.3 -> 0.00 mm
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